Commit message: Use package://zed_description URI for ZED meshes
Resolve mesh paths via the zed_description package instead of
file://$(find zed_msgs), so robot_state_publisher/RViz locate the
STL meshes correctly.

Co-Authored-By: Claude Opus 4.8 (1M context) <noreply@anthropic.com>

File: zed_wrapper/urdf/zed_macro.urdf.xacro (robot description, xacro)
@@ -172,5 +172,5 @@
           <origin xyz="${screw_offset_x} 0 ${screw_offset_z}" rpy="0 0 0"/>
           <geometry>
-            <mesh filename="file://$(find zed_msgs)/meshes/${model}.stl"/>
+            <mesh filename="package://zed_description/meshes/${model}.stl"/>
           </geometry>
             <material name="zed_mat">
@@ -181,5 +181,5 @@
           <origin xyz="${screw_offset_x} 0 ${screw_offset_z}" rpy="0 0 0"/>
           <geometry>
-            <mesh filename="file://$(find zed_msgs)/meshes/${model}.stl"/>
+            <mesh filename="package://zed_description/meshes/${model}.stl"/>
           </geometry>
         </collision>
@@ -198,5 +198,5 @@
             <origin xyz="0 0 0" rpy="0 0 0"/>
             <geometry>
-              <mesh filename="file://$(find zed_msgs)/meshes/${model}.stl"/>
+              <mesh filename="package://zed_description/meshes/${model}.stl"/>
             </geometry>
             <material name="zed_mat">
@@ -207,5 +207,5 @@
             <origin xyz="0 0 0" rpy="0 0 0"/>
             <geometry>
-              <mesh filename="file://$(find zed_msgs)/meshes/${model}.stl"/>
+              <mesh filename="package://zed_description/meshes/${model}.stl"/>
             </geometry>
           </collision>
@@ -229,5 +229,5 @@
             <origin xyz="0 0 0" rpy="0 0 0"/>
             <geometry>
-              <mesh filename="file://$(find zed_msgs)/meshes/${model}.stl"/>
+              <mesh filename="package://zed_description/meshes/${model}.stl"/>
             </geometry>
             <material name="zed_mat">
@@ -238,5 +238,5 @@
             <origin xyz="0 0 0" rpy="0 0 0"/>
             <geometry>
-              <mesh filename="file://$(find zed_msgs)/meshes/${model}.stl"/>
+              <mesh filename="package://zed_description/meshes/${model}.stl"/>
             </geometry>
           </collision>
